File: controllerpcb/controllerpcb.kicad_sch (KiCad schematic)
At the start: 29 parts

Commit message: pcb v1
Parts:
- added C1, C2, C3, C4: 0.1uF, Capacitor_SMD:C_0603_1608Metric, symbol Device:C
- added C5, C6: 100uF, Capacitor_SMD:CP_Elec_6.3x5.2, symbol Device:C_Polarized
- added F1: Polyfuse, Fuse:Fuse_1812_4532Metric, symbol Device:Polyfuse
- added J2: Screw_Terminal_01x02, TerminalBlock_Phoenix:TerminalBlock_Phoenix_MKDS-1,5-2_1x02_P5.00mm_Horizontal, symbol Connector:Screw_Terminal_01x02
- added J4, J6: Screw_Terminal_01x03, TerminalBlock_Phoenix:TerminalBlock_Phoenix_MPT-0,5-3-2.54_1x03_P2.54mm_Horizontal, symbol Connector:Screw_Terminal_01x03
- added J7: Screw_Terminal_01x08, TerminalBlock_Phoenix:TerminalBlock_Phoenix_MPT-0,5-8-2.54_1x08_P2.54mm_Horizontal, symbol Connector:Screw_Terminal_01x08
- J1: renamed from J?; mpn (none) -> 61201621621
- J3, J5: renamed from J?; mpn (none) -> B5B-XH-A(LF)(SN)
- U1, U2: renamed from U?; footprint (none) -> Package_SO:SOIC-14_3.9x8.7mm_P1.27mm
- U3, U4: renamed from U?; footprint (none) -> Package_SO:SOIC-16_3.9x9.9mm_P1.27mm; mpn (none) -> CD74HC194M
- gave numbers to parts that had none: 14
Connections:
- net +5V: now also J3.5 (Pin_5), J5.5 (Pin_5), C1.1, C2.1, C3.1, C4.1, C5.1, C6.1, F1.1, J4.3 (Pin_3), J6.3 (Pin_3)
- net GND: now also C1.2, C2.2, C3.2, C4.2, C5.2, C6.2, J2.2 (Pin_2), J7.2 (Pin_2), J7.4 (Pin_4), J7.6 (Pin_6), J7.8 (Pin_8)
- net end_a1: now also J7.1 (Pin_1)
- net end_a2: now also J7.5 (Pin_5)
- net end_b1: now also J7.3 (Pin_3)
- net end_b2: now also J7.7 (Pin_7)
- net at J5.1 (Pin_1): now also U6.16 (O1)
- net at J5.2 (Pin_2): now also U6.15 (O2)
- net at J5.3 (Pin_3): now also U6.14 (O3)
- net at J5.4 (Pin_4): now also U6.13 (O4)
- net reset2: now reaches J1.10 (Pin_10)
- net reset2: now also U4.1 (Mr)
- net dir_a2: now reaches J1.11 (Pin_11)
- net dir_a2: now also U1.13, U2.10
- net dir_b2: now reaches J1.12 (Pin_12)
- net dir_b2: now also U1.10, U2.12
- net at U4.15 (Q0), U6.1 (I1): now also U4.7 (Dsl)
- net at U6.11 (O6): now also J6.2 (Pin_2)
- net at U6.12 (O5): now also J6.1 (Pin_1)
- net at U4.12 (Q3), U6.4 (I4): now also U4.2 (Dsr)
- net at U3.15 (Q0), U5.1 (I1): now also U3.7 (Dsl)
- net at U5.11 (O6): now also J4.2 (Pin_2)
- net at U5.12 (O5): now also J4.1 (Pin_1)
- net at U5.13 (O4): now also J3.4 (Pin_4)
- net at U5.14 (O3): now also J3.3 (Pin_3)
- net at U5.15 (O2): now also J3.2 (Pin_2)
- net at U5.16 (O1): now also J3.1 (Pin_1)
- net at U3.12 (Q3), U5.4 (I4): now also U3.2 (Dsr)
- net dir_a renamed dir_a1
- net dir_a1: no longer U1.13, U2.10
- net dir_b renamed dir_b1
- net dir_b1: no longer U1.10, U2.12
- net reset renamed reset1
- net reset1: no longer U4.1 (Mr)
- new net: F1.2, J2.1 (Pin_1)
Other:
- moved on the sheet: J3, J5
